File: Hardware/v4/HeatpumpMonitor.sch (EAGLE design)
At the start: 90 parts, among them CN1 AC 9V, IC1 ATMEGA 328, Q1 BC337, Q2 BC337, T1 BC307, U1 AP2112

Commit message: Tidying up and track alignments
Connections:
- new net ESP_PUSH: U$1.GPIO2, U$2.2
- new net N$14: U$1.GPIO5
- new net N$17: U$1.GPIO4
- net RESET: no longer U$1.GPIO13, U$2.2
Other:
- note removed: "RESET"
Changed lines of the file:
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@@
 <?xml version="1.0" encoding="utf-8"?>
 <!DOCTYPE eagle SYSTEM "eagle.dtd">
-<eagle version="7.7.0">
+<eagle version="6.6.0">
 <drawing>
 <settings>
@@
 <setting verticaltext="up"/>
 </settings>
-<grid distance="0.01" unitdist="inch" unit="inch" style="lines" multiple="1" display="no" altdistance="0.01" altunitdist="inch" altunit="inch"/>
+<grid distance="0.05" unitdist="inch" unit="inch" style="lines" multiple="1" display="no" altdistance="0.01" altunitdist="inch" altunit="inch"/>
 <layers>
 <layer number="1" name="Top" color="4" fill="1" visible="no" active="no"/>
@@
 <text x="217.17" y="92.71" size="1.778" layer="91">PVT312
 Using alternative footprint here</text>
-<text x="282.448" y="21.082" size="1.778" layer="95">RESET</text>
 </plain>
 <instances>
@@
 </instance>
 <instance part="GPIO15" gate="1" x="219.71" y="15.24" smashed="yes" rot="R180">
-<attribute name="NAME" x="214.63" y="12.7" size="1.778" layer="95"/>
+<attribute name="NAME" x="214.63" y="17.78" size="1.778" layer="95"/>
 </instance>
 <instance part="GPIO0" gate="G$1" x="203.2" y="7.62"/>
@@
 </instance>
 <instance part="C9" gate="G$1" x="133.35" y="-104.14"/>
-<instance part="U$2" gate="G$1" x="290.068" y="33.02" rot="R180"/>
-<instance part="P+11" gate="G$1" x="295.148" y="31.75"/>
+<instance part="U$2" gate="G$1" x="177.8" y="25.4" rot="R270"/>
+<instance part="P+11" gate="G$1" x="182.88" y="33.02"/>
 </instances>
 <busses>
@@
 <label x="132.08" y="-68.58" size="1.778" layer="95"/>
 </segment>
-<segment>
-<pinref part="U$2" gate="G$1" pin="2"/>
-<pinref part="U$1" gate="G$1" pin="GPIO13"/>
-<wire x1="277.368" y1="27.94" x2="277.368" y2="15.24" width="0.1524" layer="91"/>
-<wire x1="277.368" y1="15.24" x2="261.62" y2="15.24" width="0.1524" layer="91"/>
-</segment>
 </net>
 <net name="N$19" class="0">
@@
 </segment>
 <segment>
+<pinref part="U$2" gate="G$1" pin="1"/>
+<wire x1="182.88" y1="30.48" x2="182.88" y2="33.02" width="0.1524" layer="91"/>
 <pinref part="P+11" gate="G$1" pin="3.3V"/>
-<wire x1="295.148" y1="31.75" x2="295.148" y2="27.94" width="0.1524" layer="91"/>
-<pinref part="U$2" gate="G$1" pin="1"/>
 </segment>
 </net>
@@
 </segment>
 </net>
+<net name="N$14" class="0">
+<segment>
+<pinref part="U$1" gate="G$1" pin="GPIO5"/>
+<wire x1="231.14" y1="7.62" x2="226.06" y2="7.62" width="0.1524" layer="91"/>
+</segment>
+</net>
+<net name="N$17" class="0">
+<segment>
+<pinref part="U$1" gate="G$1" pin="GPIO4"/>
+<wire x1="231.14" y1="5.08" x2="226.06" y2="5.08" width="0.1524" layer="91"/>
+</segment>
+</net>
+<net name="ESP_PUSH" class="0">
+<segment>
+<pinref part="U$2" gate="G$1" pin="2"/>
+<wire x1="182.88" y1="12.7" x2="182.88" y2="7.62" width="0.1524" layer="91"/>
+<label x="180.34" y="2.54" size="1.778" layer="95" rot="R90"/>
+</segment>
+<segment>
+<pinref part="U$1" gate="G$1" pin="GPIO2"/>
+<wire x1="231.14" y1="12.7" x2="226.06" y2="12.7" width="0.1524" layer="91"/>
+<label x="220.98" y="12.7" size="1.27" layer="95"/>
+</segment>
+</net>
