File: Hardware/v4/HeatpumpMonitor.brd (EAGLE design)
At the start: 99.9 x 79.9 mm, 91 parts, among them CN1 AC 9V, IC1 ATMEGA 328, Q1 BC337, Q2 BC337, T1 BC307, U1 AP2112

Commit message: Tidying up and track alignments
Parts:
- moved R10 0.32 mm to (50.0, 21.2)
Connections:
- new net ESP_PUSH: U$1.3, U$2.P$3, U$2.P$4
- new net N$14: U$1.5
- new net N$17: U$1.6
- net RESET: no longer U$1.15, U$2.P$3, U$2.P$4
Routing:
- net RESET: track 135.5 -> 57.8 mm, vias 6 -> 0
- net ESP_PUSH: track 0.00 -> 58.1 mm, vias 0 -> 4
- net GND: track 343.2 -> 336.3 mm
- net 3.3V: track 444.1 -> 443.2 mm
- net 5V: track 210.8 -> 211.4 mm

Commit message: gerbers for v4
Routing:
- net N$39: track 18.0 -> 16.5 mm
Other:
- board text added: "HEATPUMP MONITOR v0.4 (NOV 2016)"
- board text removed: "HEATPUMP MONITOR v0.3 (AUG 2016)"
- board text removed: "RESET"
Changed lines of the file:
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@@
 <text x="73.0172" y="71.1474" size="0.8128" layer="121" font="vector" ratio="20">GND     A3   A4</text>
 <text x="54.8922" y="71.1474" size="0.8128" layer="121" font="vector" ratio="20">GND  RX  TX</text>
-<text x="11.2672" y="65.7724" size="1.27" layer="121" font="vector" ratio="20">HEATPUMP MONITOR v0.3 (AUG 2016)</text>
+<text x="11.2672" y="65.7724" size="1.27" layer="121" font="vector" ratio="20">HEATPUMP MONITOR v0.4 (NOV 2016)</text>
 <text x="11.2672" y="63.7724" size="1.27" layer="121" font="vector" ratio="20">An OpenEnergyMonitor project</text>
 <text x="9.0172" y="13.2724" size="1.27" layer="121" font="vector" ratio="20">Designed in
@@
 <wire x1="55.75" y1="15" x2="46.75" y2="15" width="0.4064" layer="46"/>
 <wire x1="46.75" y1="15" x2="46.75" y2="14.375" width="0.4064" layer="46"/>
-<text x="96.52" y="20.32" size="0.4064" layer="25">RESET</text>
 </plain>
 <attributes>
@@
 <attribute name="VALUE" x="70.722" y="12.083" size="0.8128" layer="27" font="vector" ratio="20"/>
 </element>
-<element name="R3" library="rcl" package="0204/7" value="10k" x="62.75" y="20" smashed="yes" rot="R180">
-<attribute name="NAME" x="63.636" y="21.9986" size="0.9906" layer="25" ratio="10" rot="R180"/>
-<attribute name="VALUE" x="65.8806" y="19.0856" size="0.9906" layer="27" ratio="10" rot="R180"/>
-</element>
+<element name="R3" library="rcl" package="0204/7" value="10k" x="62.75" y="20" smashed="yes" rot="R180"/>
 <element name="R8" library="rcl" package="0207/2V" value="100k" x="72.5" y="69.75" smashed="yes">
 <attribute name="NAME" x="69.734" y="69.1992" size="0.8128" layer="25" font="vector" ratio="20" rot="R90"/>
@@
 <contactref element="U$1" pad="11"/>
 <contactref element="CH_PD" pad="2"/>
-<wire x1="95.236" y1="26.474" x2="95.236" y2="25.486" width="0.4064" layer="1"/>
-<wire x1="95.236" y1="25.486" x2="93.75" y2="24" width="0.4064" layer="1"/>
-<wire x1="93.75" y1="24" x2="93.25" y2="24" width="0.4064" layer="1"/>
-<wire x1="93.25" y1="24" x2="91.742" y2="22.746" width="0.4064" layer="1"/>
-<wire x1="91.742" y1="22.746" x2="91.742" y2="13.996" width="0.4064" layer="1"/>
-<wire x1="91.742" y1="13.996" x2="94" y2="12.5" width="0.4064" layer="1"/>
+<wire x1="95.236" y1="26.474" x2="95.236" y2="25.4368" width="0.4064" layer="1"/>
 <wire x1="94" y1="12.5" x2="95" y2="12.5" width="0.4064" layer="1"/>
+<wire x1="95.236" y1="25.4368" x2="92.8116" y2="23.0124" width="0.4064" layer="1"/>
+<wire x1="92.8116" y1="23.0124" x2="92.8116" y2="13.6884" width="0.4064" layer="1"/>
+<wire x1="92.8116" y1="13.6884" x2="94" y2="12.5" width="0.4064" layer="1"/>
 </signal>
 <signal name="N$40">
