File: Hardware/WiFi_MBUS_Reader/v2/v2.sch (EAGLE design)
At the start: 33 parts, among them U1 AP2112

Commit message: new MBUS reader hardware designs
Parts:
- removed FTDI1: FTDI, JeeLabs:MA06-1
- removed JP4, JP5, JP6, JP7: (no value), SparkFun:M02PTH
- removed RX_LINK, TX_LINK: SOLDERJUMPERNO, SparkFun:SOLDERJUMPERNO
- added C1: 4.7u, SparkFun-Capacitors:1.0UF-0805-25V-(+80/-20%)
- added C2: 10u, SparkFun-Capacitors:1.0UF-1206-50V-10%
- added C3: 1u, SparkFun-Capacitors:1.0UF-1206-50V-10%
- added C6, C7: 100nF, SparkFun:CAP0603-CAP
- added CR1: CR1220SMD, IotaWatt_parts:CR1220SMD
- added D1: SS14, adafruit:DIODESOD-123
- added F1: 6V/0.5A, SparkFun-Fuses:PPTC_HALF-AMP
- added F2: PTCSMD, SparkFun:PTCSMD
- added IC2: CP210X_USB_UART, SparkFun-DigitalIC:CP210X_USB_UART
- added L1: 10uH, SparkFun:INDUCTORCR54
- added MICRO_SD: 47219-2001_MICROSD, MOLEX 47219-2001:47219-2001_MICROSD
- added R1: 1M, SparkFun-Resistors:RESISTOR0805
- added R10: 37k, SparkFun-Resistors:RESISTOR0805
- added U2: AP3015, dword1511-pmic-dcdc:AP3015
- added U3: DS3231MZ+TRL, DS3231MZ_TRL:DS3231MZ+TRL
- added U4: ESP8266-12E/ESP-12E, ESP8266-12E_ESP-12E:ESP8266-12E/ESP-12E
Connections:
- removed net ESPRX: FTDI1.3, TX_LINK.1, U$1.RXD
- removed net ESPTX: FTDI1.2, RX_LINK.1, U$1.TXD
- new net D+: IC2.D+, U$10.D+
- new net D-: IC2.D-, U$10.D-
- new net DTR: IC2.DTR
- new net GPIO12: MICRO_SD.DAT0
- new net GPIO13: MICRO_SD.CMD
- new net GPIO14: MICRO_SD.CLK
- new net GPIO15: MICRO_SD.CD/DAT3
- new net N$1: C7.1, IC2.VDD
- new net N$2: F2.1, U$10.VBUS
- new net N$4: R1.1, R10.2, U2.FB
- new net N$5: D1.A, L1.2, U2.SW
- new net N$6: CR1.P$+, U3.VBAT
- new net RXD: IC2.RXD, U$1.TXD
- new net SCL: U3.SCL
- new net SDA: U3.SDA
- new net TXD: IC2.TXD, U$1.RXD
- net 24V: now also C2.1, C3.1, D1.C, R1.2; no longer JP5.1, JP5.2
- net 3.3V: now also MICRO_SD.VDD, U3.VCC
- net 5V: now also C1.1, F1.2, L1.1, U2.EN, U2.VIN; no longer JP7.1, JP7.2
- net 5V1: now also C6.1, F1.1, F2.2, IC2.REGIN, IC2.VBUS; no longer FTDI1.4, U$10.VBUS
- net D12: no longer RX_LINK.2
- net D14: no longer TX_LINK.2
- net GND: now also C1.2, C2.2, C3.2, C6.2, C7.2, CR1.P$-, IC2.GND, IC2.GND@EXP, IC2.GND@M, MICRO_SD.GND, MICRO_SD.VSS, R10.1, U2.GND, U3.GND; no longer FTDI1.6, JP4.1, JP4.2, JP6.1, JP6.2
Other:
- note added: "MICRO SD CARD"
- moved on the sheet: C20, C21, U1
