File: Hardware/USB_to_MBUS/USB_to_MBUS.brd (EAGLE design)
At the start: 24 x 42 mm, 30 parts, among them CN1 1X4-BIG, IC2 CP210X_USB_UART, J1 1X2-3.5MM, U2 AP3015

Commit message: heat pump monitor Pi base board and latest USB to MBUS reader
Parts:
- removed J1: 1X2-3.5MM, adafruit:1X2-3.5MM
- added CN2: 1X4-3.5MM, adafruit:1X04-3.5MM
- moved R17 2.32 mm to (20.3, 34.6)
- moved C3 0.30 mm to (5.49, 34.4)
Connections:
- net 24V: now also CN2.3, CN2.4; no longer J1.1
- net N$13: now also CN2.1, CN2.2; no longer J1.2
Routing:
- net 24V: track 31.7 -> 37.0 mm
- net N$13: track 11.3 -> 12.0 mm
