File: Hardware/USB_to_MBUS/USB_to_MBUS.sch (EAGLE design)
At the start: 29 parts, among them CN1 1X4-BIG, IC2 CP210X_USB_UART, J1 1X2-3.5MM, U2 AP3015

Commit message: heat pump monitor Pi base board and latest USB to MBUS reader
Parts:
- removed J1: 1X2-3.5MM, adafruit:1X2-3.5MM
- added CN2: 1X4-3.5MM, adafruit:1X4-3.5MM
Connections:
- net 24V: now also CN2.3, CN2.4; no longer J1.1
- net N$13: now also CN2.1, CN2.2; no longer J1.2
